File: CADs/HoneyVendingCompleteBoard/HoneyVendingCompleteBoard.sch (KiCad schematic (older format))
At the start: 16 parts, among them J1 SegmentPins, J2 CoinPins, J3 ConnToDoors, J4 12V Power, J6 Conn_01x05_Male, U1 L7805

Commit message: Split Main Board into Main Board and Button Board
Parts:
- removed J6: Conn_01x05_Male, Connector_PinHeader_2.54mm:PinHeader_1x05_P2.54mm_Vertical, symbol Connector:Conn_01x05_Male
- added 100nF2: ButtonDecouple, Capacitor_THT:C_Disc_D6.0mm_W2.5mm_P5.00mm, symbol Device:C
- added 100nF3: ButtonC, Capacitor_THT:C_Disc_D6.0mm_W2.5mm_P5.00mm, symbol Device:C
- added 10kOhm3: R, Resistor_SMD:R_0805_2012Metric_Pad1.15x1.40mm_HandSolder, symbol Device:R
- added 10kOhm4: ButtonR4, Resistor_SMD:R_0805_2012Metric_Pad1.15x1.40mm_HandSolder, symbol Device:R
- added 10kOhm5: ButtonR5, Resistor_SMD:R_0805_2012Metric_Pad1.15x1.40mm_HandSolder, symbol Device:R
- added 10kOhm6: ButtonR6, Resistor_SMD:R_0805_2012Metric_Pad1.15x1.40mm_HandSolder, symbol Device:R
- added 10kOhm7: ButtonR2, Resistor_SMD:R_0805_2012Metric_Pad1.15x1.40mm_HandSolder, symbol Device:R
- added 10kOhm8: ButtonR3, Resistor_SMD:R_0805_2012Metric_Pad1.15x1.40mm_HandSolder, symbol Device:R
- added 10kOhm9: ButtonR1, Resistor_SMD:R_0805_2012Metric_Pad1.15x1.40mm_HandSolder, symbol Device:R
- added Button1, Button2, Button3, Button4, Button5, Button6: SW_DPST_x2, Button_Switch_THT:SW_PUSH_6mm_H9.5mm, symbol Switch:SW_DPST_x2
- added J5: Power Line, Connector_PinHeader_2.54mm:PinHeader_1x02_P2.54mm_Vertical, symbol Connector_Generic:Conn_01x02
- added U2: 74HC165, Customs:74HC165, symbol 74xx:74HC165
Connections:
- wire segments 94 -> 165
Other:
- note added: "SER\nSRCLK\nSRCLR\nRCLK\nOE\n+5V\nUnconn\nUnconn"
- note removed: "5V\nButtonShift/Load\nButtonClock\nButtonSEROutput\nGND\n"
- note removed: "SER\nSRCLK\nSRCLR\nRCLK\nOE\n+5V\nGND\n12V"
